File: skidl/pcb/solartron_7075_interface.kicad_pcb (KiCad board)
At the start: 4 copper layers, 112 x 44 mm, 94 parts, among them J1 DD-50 plug, J2 USB_B, J3 SWD, Q1 2N7002, SW1 BOOTSEL, SW2 RESET, U1 RP2354A, U10 74HCT165, U11 74HCT165, U12 74HCT165, U13 74HCT165, U14 74HCT165, U15 74HC595, U16 74HC595, U2 AP2112K-3.3, U3 USBLC6-2SC6, U4 78L05, U5 TLP2361, U6 TLP2361, U7 TLP2361, U8 TLP2361, U9 TLP2361, Y1 12MHz

Commit message: Add verified single-page schematic, link board to it, split README issues
- scripts/gen_schematic.py draws one A2 sheet from the SKiDL netlist
  (SKiDL's own generator mis-connects nets on this design) and checks it by
  re-exporting the netlist with kicad-cli: all 135 nets match in pins and
  names. KiCad ERC: 0 violations.
- scripts/link_schematic.py gives footprints their symbol paths and BOM
  fields, renames nets as KiCad's Update PCB would, and adds no-connect
  nets, so DRC with --schematic-parity is clean (0/0/0). Copper unchanged.
- build.sh runs both steps and exports the schematic PDF/PNG.
- README: schematic section; tool issues separated from design caveats.

Co-Authored-By: Claude Opus 5.5 <noreply@anthropic.com>
Claude-Session: https://claude.ai/code/session_01ERGgANCwEg9niX4WLDjBj2
Connections:
- net AUTORANGE_INH renamed /AUTORANGE_INH
- net BCD_1E0_1 renamed /BCD_1E0_1
- net BCD_1E0_1_R renamed /BCD_1E0_1_R
- net BCD_1E0_2 renamed /BCD_1E0_2
- net BCD_1E0_2_R renamed /BCD_1E0_2_R
- net BCD_1E0_4 renamed /BCD_1E0_4
- net BCD_1E0_4_R renamed /BCD_1E0_4_R
- net BCD_1E0_8 renamed /BCD_1E0_8
- net BCD_1E0_8_R renamed /BCD_1E0_8_R
- net BCD_1E1_1 renamed /BCD_1E1_1
- net BCD_1E1_1_R renamed /BCD_1E1_1_R
- net BCD_1E1_2 renamed /BCD_1E1_2
- net BCD_1E1_2_R renamed /BCD_1E1_2_R
- net BCD_1E1_4 renamed /BCD_1E1_4
- net BCD_1E1_4_R renamed /BCD_1E1_4_R
- net BCD_1E1_8 renamed /BCD_1E1_8
- net BCD_1E1_8_R renamed /BCD_1E1_8_R
- net BCD_1E2_1 renamed /BCD_1E2_1
- net BCD_1E2_1_R renamed /BCD_1E2_1_R
- net BCD_1E2_2 renamed /BCD_1E2_2
- net BCD_1E2_2_R renamed /BCD_1E2_2_R
- net BCD_1E2_4 renamed /BCD_1E2_4
- net BCD_1E2_4_R renamed /BCD_1E2_4_R
- net BCD_1E2_8 renamed /BCD_1E2_8
- net BCD_1E2_8_R renamed /BCD_1E2_8_R
- net BCD_1E3_1 renamed /BCD_1E3_1
- net BCD_1E3_1_R renamed /BCD_1E3_1_R
- net BCD_1E3_2 renamed /BCD_1E3_2
- net BCD_1E3_2_R renamed /BCD_1E3_2_R
- net BCD_1E3_4 renamed /BCD_1E3_4
- net BCD_1E3_4_R renamed /BCD_1E3_4_R
- net BCD_1E3_8 renamed /BCD_1E3_8
- net BCD_1E3_8_R renamed /BCD_1E3_8_R
- net BCD_1E4_1 renamed /BCD_1E4_1
- net BCD_1E4_1_R renamed /BCD_1E4_1_R
- net BCD_1E4_2 renamed /BCD_1E4_2
- net BCD_1E4_2_R renamed /BCD_1E4_2_R
- net BCD_1E4_4 renamed /BCD_1E4_4
- net BCD_1E4_4_R renamed /BCD_1E4_4_R
- net BCD_1E4_8 renamed /BCD_1E4_8
- net BCD_1E4_8_R renamed /BCD_1E4_8_R
- net BCD_1E5_1 renamed /BCD_1E5_1
- net BCD_1E5_1_R renamed /BCD_1E5_1_R
- net BCD_1E5_2 renamed /BCD_1E5_2
- net BCD_1E5_2_R renamed /BCD_1E5_2_R
- net BCD_1E5_4 renamed /BCD_1E5_4
- net BCD_1E5_4_R renamed /BCD_1E5_4_R
- net BCD_1E5_8 renamed /BCD_1E5_8
- net BCD_1E5_8_R renamed /BCD_1E5_8_R
- net BCD_1E6_1 renamed /BCD_1E6_1
- net BCD_1E6_1_R renamed /BCD_1E6_1_R
- net BOOTSEL renamed /BOOTSEL
- net DATA_CAN_CHANGE renamed /DATA_CAN_CHANGE
- net DATA_CAN_CHANGE_R renamed /DATA_CAN_CHANGE_R
- net FUNC_CMD_42 renamed /FUNC_CMD_42
- net FUNC_CMD_43 renamed /FUNC_CMD_43
- net FUNC_OUT_A renamed /FUNC_OUT_A
- net FUNC_OUT_A_R renamed /FUNC_OUT_A_R
- net FUNC_OUT_B renamed /FUNC_OUT_B
- net FUNC_OUT_B_R renamed /FUNC_OUT_B_R
- net INTEG_1 renamed /INTEG_1
- net INTEG_2 renamed /INTEG_2
- net INTEG_4 renamed /INTEG_4
- net ISO_LATCH renamed /ISO_LATCH
- net ISO_MISO_K renamed /ISO_MISO_K
- net ISO_MOSI renamed /ISO_MOSI
- net ISO_OE_N renamed /ISO_OE_N
- net ISO_SCLK renamed /ISO_SCLK
- net LED_ISO_PWR_A renamed /LED_ISO_PWR_A
- net LED_PWR_A renamed /LED_PWR_A
- net LED_REMOTE renamed /LED_REMOTE
- net LED_REMOTE_A renamed /LED_REMOTE_A
- net LED_STATUS renamed /LED_STATUS
- net LED_STATUS_A renamed /LED_STATUS_A
- net LOCKOUT_N renamed /LOCKOUT_N
- net MCU_LATCH renamed /MCU_LATCH
- net MCU_MISO renamed /MCU_MISO
- net MCU_MOSI renamed /MCU_MOSI
- net MCU_OE_N renamed /MCU_OE_N
- net MCU_SCLK renamed /MCU_SCLK
- net MCU_USB_DM renamed /MCU_USB_DM
- net MCU_USB_DP renamed /MCU_USB_DP
- net OVERLOAD renamed /OVERLOAD
- net OVERLOAD_R renamed /OVERLOAD_R
- net POL_NEG renamed /POL_NEG
- net POL_NEG_R renamed /POL_NEG_R
- net POL_POS renamed /POL_POS
- net POL_POS_R renamed /POL_POS_R
- net PRINT_LEVEL renamed /PRINT_LEVEL
- net PRINT_LEVEL_R renamed /PRINT_LEVEL_R
- net PRINT_PULSE renamed /PRINT_PULSE
- net PRINT_PULSE_R renamed /PRINT_PULSE_R
- net QSPI_SS renamed /QSPI_SS
- net RANGE_CMD_1 renamed /RANGE_CMD_1
- net RANGE_CMD_2 renamed /RANGE_CMD_2
- net RANGE_CMD_4 renamed /RANGE_CMD_4
- net RANGE_OUT_1 renamed /RANGE_OUT_1
- net RANGE_OUT_1_R renamed /RANGE_OUT_1_R
- net RANGE_OUT_2 renamed /RANGE_OUT_2
- net RANGE_OUT_2_R renamed /RANGE_OUT_2_R
- net RANGE_OUT_4 renamed /RANGE_OUT_4
- net RANGE_OUT_4_R renamed /RANGE_OUT_4_R
- net RATIO_N renamed /RATIO_N
- net RUN renamed /RUN
- net SAMPLE_CONTACT renamed /SAMPLE_CONTACT
- net SAMPLE_CONTACT_DRV renamed /SAMPLE_CONTACT_DRV
- net SAMPLE_PULSE renamed /SAMPLE_PULSE
- net SR165_CHAIN1 renamed /SR165_CHAIN1
- net SR165_CHAIN2 renamed /SR165_CHAIN2
- net SR165_CHAIN3 renamed /SR165_CHAIN3
- net SR165_CHAIN4 renamed /SR165_CHAIN4
- net SR595_CHAIN renamed /SR595_CHAIN
- net SWCLK renamed /SWCLK
- net SWDIO renamed /SWDIO
- net U5_A renamed /U5_A
- net U6_A renamed /U6_A
- net U7_A renamed /U7_A
- net U8_A renamed /U8_A
- net U9_A renamed /U9_A
- net USB_D+ renamed /USB_D+
- net USB_D- renamed /USB_D-
- net USB_SHIELD renamed /USB_SHIELD
- net VBUS_RAW renamed /VBUS_RAW
- net VREG_AVDD renamed /VREG_AVDD
- net VREG_LX renamed /VREG_LX
- net XIN renamed /XIN
- net XOUT renamed /XOUT
- net XOUT_R renamed /XOUT_R
- U1 pad 10: (no net) -> unconnected-(U1-GPIO7-Pad10)
- U1 pad 12: (no net) -> unconnected-(U1-GPIO8-Pad12)
- U1 pad 13: (no net) -> unconnected-(U1-GPIO9-Pad13)
- U1 pad 14: (no net) -> unconnected-(U1-GPIO10-Pad14)
- U1 pad 15: (no net) -> unconnected-(U1-GPIO11-Pad15)
- U1 pad 16: (no net) -> unconnected-(U1-GPIO12-Pad16)
- U1 pad 17: (no net) -> unconnected-(U1-GPIO13-Pad17)
- U1 pad 18: (no net) -> unconnected-(U1-GPIO14-Pad18)
- U1 pad 19: (no net) -> unconnected-(U1-GPIO15-Pad19)
- U1 pad 2: (no net) -> unconnected-(U1-GPIO0-Pad2)
- U1 pad 27: (no net) -> unconnected-(U1-GPIO16-Pad27)
- U1 pad 28: (no net) -> unconnected-(U1-GPIO17-Pad28)
- U1 pad 29: (no net) -> unconnected-(U1-GPIO18-Pad29)
- U1 pad 3: (no net) -> unconnected-(U1-GPIO1-Pad3)
- U1 pad 31: (no net) -> unconnected-(U1-GPIO19-Pad31)
- U1 pad 37: (no net) -> unconnected-(U1-GPIO25-Pad37)
- U1 pad 4: (no net) -> unconnected-(U1-GPIO2-Pad4)
- U1 pad 40: (no net) -> unconnected-(U1-GPIO26/ADC0-Pad40)
- U1 pad 41: (no net) -> unconnected-(U1-GPIO27/ADC1-Pad41)
- U1 pad 42: (no net) -> unconnected-(U1-GPIO28/ADC2-Pad42)
- U1 pad 43: (no net) -> unconnected-(U1-GPIO29/ADC3-Pad43)
- U1 pad 5: (no net) -> unconnected-(U1-GPIO3-Pad5)
- U1 pad 55: (no net) -> unconnected-(U1-QSPI_SD3-Pad55)
- U1 pad 56: (no net) -> unconnected-(U1-QSPI_SCLK-Pad56)
- U1 pad 57: (no net) -> unconnected-(U1-QSPI_SD0-Pad57)
- U1 pad 58: (no net) -> unconnected-(U1-QSPI_SD2-Pad58)
- U1 pad 59: (no net) -> unconnected-(U1-QSPI_SD1-Pad59)
- U1 pad 7: (no net) -> unconnected-(U1-GPIO4-Pad7)
- U1 pad 9: (no net) -> unconnected-(U1-GPIO6-Pad9)
- U10 pad 7: (no net) -> unconnected-(U10-~{Q7}-Pad7)
- U11 pad 7: (no net) -> unconnected-(U11-~{Q7}-Pad7)
- U12 pad 7: (no net) -> unconnected-(U12-~{Q7}-Pad7)
- U13 pad 7: (no net) -> unconnected-(U13-~{Q7}-Pad7)
- U14 pad 7: (no net) -> unconnected-(U14-~{Q7}-Pad7)
- U16 pad 6: (no net) -> unconnected-(U16-QG-Pad6)
- U16 pad 7: (no net) -> unconnected-(U16-QH-Pad7)
- U16 pad 9: (no net) -> unconnected-(U16-QH'-Pad9)
- U2 pad 4: (no net) -> unconnected-(U2-NC-Pad4)
