File: skidl/pcb/solartron_7075_interface.kicad_sch (KiCad schematic)
At the start: 94 parts, among them J1 DD-50 plug, J2 USB_B, J3 SWD, Q1 2N7002, SW1 BOOTSEL, SW2 RESET, U1 RP2354A, U10 74HCT165, U11 74HCT165, U12 74HCT165, U13 74HCT165, U14 74HCT165, U15 74HC595, U16 74HC595, U2 AP2112K-3.3, U3 USBLC6-2SC6, U4 78L05, U5 TLP2361, U6 TLP2361, U7 TLP2361, U8 TLP2361, U9 TLP2361, Y1 12MHz

Commit message: skidl: tidy meter-side routing by pin swapping within parts
Reassign the D inputs of the 74HCT165s (U14's link-check inputs included),
the channels of the resistor arrays and the outputs of the 74HC595s, found by
scripts/optimise_pins.py (simulated annealing on straight-line crossings and
length; no part moved, no signal moved to another part). Re-routed with
Freerouting:

  arrays -> 74HCT165s: 64 -> 0 crossings, 441 -> 351 mm of track
  74HC595s -> J1:      36 -> 8 crossings, 265 -> 205 mm
  J1 -> arrays:       148 -> 102 crossings, 513 -> 481 mm
  whole board:        2428 -> 2227 mm of track, 262 -> 260 vias

DRC, ERC and schematic parity remain clean. The bit maps in the README and
the schematic notes (now generated from the netlist) follow the new
assignment; the link-check pattern is now 0011 on U14 D5..D2.

Co-Authored-By: Claude Opus 5.5 <noreply@anthropic.com>
Claude-Session: https://claude.ai/code/session_01ERGgANCwEg9niX4WLDjBj2
Connections:
- net AUTORANGE_INH: now also U15.15 (QA); no longer U15.7 (QH)
- net BCD_1E0_1: now also RN8.1 (R1.1); no longer RN8.4 (R4.1)
- net BCD_1E0_1_R: now also RN8.8 (R1.2), U13.5 (D6); no longer RN8.5 (R4.2), U13.11 (D0)
- net BCD_1E0_2: now also RN8.2 (R2.1); no longer RN8.3 (R3.1)
- net BCD_1E0_2_R: now also RN8.7 (R2.2), U13.4 (D5); no longer RN8.6 (R3.2), U13.12 (D1)
- net BCD_1E0_4: now also RN8.3 (R3.1); no longer RN8.2 (R2.1)
- net BCD_1E0_4_R: now also RN8.6 (R3.2), U13.3 (D4); no longer RN8.7 (R2.2), U13.13 (D2)
- net BCD_1E0_8: now also RN8.4 (R4.1); no longer RN8.1 (R1.1)
- net BCD_1E0_8_R: now also RN8.5 (R4.2), U13.6 (D7); no longer RN8.8 (R1.2), U13.14 (D3)
- net BCD_1E1_1: now also RN7.1 (R1.1); no longer RN7.4 (R4.1)
- net BCD_1E1_1_R: now also RN7.8 (R1.2), U13.11 (D0); no longer RN7.5 (R4.2), U13.3 (D4)
- net BCD_1E1_2: now also RN7.2 (R2.1); no longer RN7.3 (R3.1)
- net BCD_1E1_2_R: now also RN7.7 (R2.2), U13.13 (D2); no longer RN7.6 (R3.2), U13.4 (D5)
- net BCD_1E1_4: now also RN7.3 (R3.1); no longer RN7.2 (R2.1)
- net BCD_1E1_4_R: now also RN7.6 (R3.2), U13.14 (D3); no longer RN7.7 (R2.2), U13.5 (D6)
- net BCD_1E1_8: now also RN7.4 (R4.1); no longer RN7.1 (R1.1)
- net BCD_1E1_8_R: now also RN7.5 (R4.2), U13.12 (D1); no longer RN7.8 (R1.2), U13.6 (D7)
- net BCD_1E2_1: now also RN4.1 (R1.1); no longer RN4.4 (R4.1)
- net BCD_1E2_1_R: now also RN4.8 (R1.2), U11.5 (D6); no longer RN4.5 (R4.2), U11.11 (D0)
- net BCD_1E2_2: now also RN4.2 (R2.1); no longer RN4.3 (R3.1)
- net BCD_1E2_2_R: now also RN4.7 (R2.2), U11.4 (D5); no longer RN4.6 (R3.2), U11.12 (D1)
- net BCD_1E2_4: now also RN4.3 (R3.1); no longer RN4.2 (R2.1)
- net BCD_1E2_4_R: now also RN4.6 (R3.2), U11.3 (D4); no longer RN4.7 (R2.2), U11.13 (D2)
- net BCD_1E2_8: now also RN4.4 (R4.1); no longer RN4.1 (R1.1)
- net BCD_1E2_8_R: now also RN4.5 (R4.2), U11.6 (D7); no longer RN4.8 (R1.2), U11.14 (D3)
- net BCD_1E3_1: now also RN3.1 (R1.1); no longer RN3.4 (R4.1)
- net BCD_1E3_1_R: now also RN3.8 (R1.2), U11.11 (D0); no longer RN3.5 (R4.2), U11.3 (D4)
- net BCD_1E3_2: now also RN3.2 (R2.1); no longer RN3.3 (R3.1)
- net BCD_1E3_2_R: now also RN3.7 (R2.2), U11.13 (D2); no longer RN3.6 (R3.2), U11.4 (D5)
- net BCD_1E3_4: now also RN3.3 (R3.1); no longer RN3.2 (R2.1)
- net BCD_1E3_4_R: now also RN3.6 (R3.2), U11.14 (D3); no longer RN3.7 (R2.2), U11.5 (D6)
- net BCD_1E3_8: now also RN3.4 (R4.1); no longer RN3.1 (R1.1)
- net BCD_1E3_8_R: now also RN3.5 (R4.2), U11.12 (D1); no longer RN3.8 (R1.2), U11.6 (D7)
- net BCD_1E4_1: now also RN6.1 (R1.1); no longer RN6.4 (R4.1)
- net BCD_1E4_1_R: now also RN6.8 (R1.2), U12.6 (D7); no longer RN6.5 (R4.2), U12.11 (D0)
- net BCD_1E4_2: now also RN6.2 (R2.1); no longer RN6.3 (R3.1)
- net BCD_1E4_2_R: now also RN6.7 (R2.2), U12.3 (D4); no longer RN6.6 (R3.2), U12.12 (D1)
- net BCD_1E4_4: now also RN6.3 (R3.1); no longer RN6.2 (R2.1)
- net BCD_1E4_4_R: now also RN6.6 (R3.2), U12.4 (D5); no longer RN6.7 (R2.2), U12.13 (D2)
- net BCD_1E4_8: now also RN6.4 (R4.1); no longer RN6.1 (R1.1)
- net BCD_1E4_8_R: now also RN6.5 (R4.2), U12.5 (D6); no longer RN6.8 (R1.2), U12.14 (D3)
- net BCD_1E5_1: now also RN5.1 (R1.1); no longer RN5.4 (R4.1)
- net BCD_1E5_1_R: now also RN5.8 (R1.2), U12.11 (D0); no longer RN5.5 (R4.2), U12.3 (D4)
- net BCD_1E5_2: now also RN5.2 (R2.1); no longer RN5.3 (R3.1)
- net BCD_1E5_2_R: now also RN5.7 (R2.2), U12.14 (D3); no longer RN5.6 (R3.2), U12.4 (D5)
- net BCD_1E5_4: now also RN5.3 (R3.1); no longer RN5.2 (R2.1)
- net BCD_1E5_4_R: now also RN5.6 (R3.2), U12.13 (D2); no longer RN5.7 (R2.2), U12.5 (D6)
- net BCD_1E5_8: now also RN5.4 (R4.1); no longer RN5.1 (R1.1)
- net BCD_1E5_8_R: now also RN5.5 (R4.2), U12.12 (D1); no longer RN5.8 (R1.2), U12.6 (D7)
- net BCD_1E6_1: now also RN9.2 (R2.1); no longer RN9.4 (R4.1)
- net BCD_1E6_1_R: now also RN9.7 (R2.2), U14.5 (D6); no longer RN9.5 (R4.2), U14.3 (D4)
- net DATA_CAN_CHANGE: now also RN9.3 (R3.1); no longer RN9.2 (R2.1)
- net DATA_CAN_CHANGE_R: now also RN9.6 (R3.2), U14.11 (D0); no longer RN9.7 (R2.2), U14.5 (D6)
- net FUNC_CMD_42: now also U15.5 (QF); no longer U15.2 (QC)
- net FUNC_CMD_43: now also U15.4 (QE); no longer U15.3 (QD)
- net FUNC_OUT_A: now also RN1.2 (R2.1); no longer RN1.3 (R3.1)
- net FUNC_OUT_A_R: now also RN1.7 (R2.2), U10.13 (D2); no longer RN1.6 (R3.2), U10.4 (D5)
- net FUNC_OUT_B: now also RN1.1 (R1.1); no longer RN1.4 (R4.1)
- net FUNC_OUT_B_R: now also RN1.8 (R1.2), U10.12 (D1); no longer RN1.5 (R4.2), U10.3 (D4)
- net INTEG_1: now also U15.1 (QB); no longer U15.4 (QE)
- net INTEG_2: now also U15.2 (QC); no longer U15.5 (QF)
- net INTEG_4: now also U15.3 (QD); no longer U15.6 (QG)
- net ISO_+5V: now also U14.13 (D2); no longer U14.12 (D1)
- net ISO_GND: now also U14.3 (D4), U14.4 (D5); no longer U14.11 (D0), U14.13 (D2)
- net LED_REMOTE: now also U16.15 (QA); no longer U16.5 (QF)
- net LOCKOUT_N: now also U15.7 (QH); no longer U15.15 (QA)
- net OVERLOAD: now also RN9.4 (R4.1); no longer RN9.3 (R3.1)
- net OVERLOAD_R: now also RN9.5 (R4.2), U14.12 (D1); no longer RN9.6 (R3.2), U14.4 (D5)
- net POL_NEG: now also RN1.3 (R3.1); no longer RN1.2 (R2.1)
- net POL_NEG_R: now also RN1.6 (R3.2), U10.14 (D3); no longer RN1.7 (R2.2), U10.5 (D6)
- net POL_POS: now also RN1.4 (R4.1); no longer RN1.1 (R1.1)
- net POL_POS_R: now also RN1.5 (R4.2), U10.11 (D0); no longer RN1.8 (R1.2), U10.6 (D7)
- net PRINT_PULSE: now also RN2.1 (R1.1); no longer RN2.4 (R4.1)
- net PRINT_PULSE_R: now also RN2.8 (R1.2), U10.4 (D5); no longer RN2.5 (R4.2), U10.11 (D0)
- net RANGE_CMD_1: now also U16.7 (QH); no longer U16.15 (QA)
- net RANGE_CMD_2: now also U16.5 (QF); no longer U16.1 (QB)
- net RANGE_CMD_4: now also U16.4 (QE); no longer U16.2 (QC)
- net RANGE_OUT_1: now also RN2.2 (R2.1); no longer RN2.3 (R3.1)
- net RANGE_OUT_1_R: now also RN2.7 (R2.2), U10.3 (D4); no longer RN2.6 (R3.2), U10.12 (D1)
- net RANGE_OUT_2: now also RN2.3 (R3.1); no longer RN2.2 (R2.1)
- net RANGE_OUT_2_R: now also RN2.6 (R3.2), U10.5 (D6); no longer RN2.7 (R2.2), U10.13 (D2)
- net RANGE_OUT_4: now also RN2.4 (R4.1); no longer RN2.1 (R1.1)
- net RANGE_OUT_4_R: now also RN2.5 (R4.2), U10.6 (D7); no longer RN2.8 (R1.2), U10.14 (D3)
- net RATIO_N: now also U15.6 (QG); no longer U15.1 (QB)
- net SAMPLE_CONTACT_DRV: now also U16.3 (QD); no longer U16.4 (QE)
- net SAMPLE_PULSE: now also U16.6 (QG); no longer U16.3 (QD)
Other:
- note added: "Isolated serial link (RP2354A SPI0 / PIO): SPI mode 0, MSB first, <= 1 MHz, 40 clocks per transfer. Pulse LATCH low >= 1 us, then clock 5 bytes. LATCH low: the 74HCT165s sample the meter outputs. LATCH rising edge: the 74HC595 outputs take the last two bytes clocked in. /OE (GPIO24) high = command outputs off (the default while the MCU is unpowered or in reset). MISO byte0 U10: RANGE_4 RANGE_2 PR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"
- note removed: "Isolated serial link (RP2354A SPI0 / PIO): SPI mode 0, MSB first, <= 1 MHz, 40 clocks per transfer. Pulse LATCH low >= 1 us, then clock 5 bytes. LATCH low: the 74HCT165s sample the meter outputs. LATCH rising edge: the 74HC595 outputs take the last two bytes clocked in. /OE (GPIO24) high = command outputs off (the default while the MCU is unpowered or in reset). MISO byte0 U10: POL+ POL- FUNC_A F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"

Commit message: skidl: swap pins between parts and move the meter-side registers
scripts/optimise_layout.py extends the pin-swap search across parts (any
meter output on any array channel and 74HCT165 input, any command input on
any 74HC595 output) and lets the registers change places and turn 180
degrees; it also scores the clock, latch, /OE, MOSI and chain nets. Result:
all seven registers turned 180 degrees (control and supply pins away from J1
and the arrays), the 74HCT165s in chain order along the bottom row, U15/U16
swapped, decoupling caps moved with the supply pins. Re-routed:

  J1 -> arrays:     102 -> 10 crossings, 481 -> 255 mm of track, 18 -> 6 vias
  74HC595s -> J1:     8 -> 1 crossing,   205 -> 137 mm, 11 -> 7 vias
  control + chains:                      558 -> 494 mm
  whole board:      2227 -> 1868 mm of track, 260 -> 243 vias

DRC, ERC and schematic parity are clean. README bit maps and the routing
review section are updated; the link check is now 1010 on U14 D3..D0.

Co-Authored-By: Claude Opus 5.5 <noreply@anthropic.com>
Claude-Session: https://claude.ai/code/session_01ERGgANCwEg9niX4WLDjBj2
Connections:
- net AUTORANGE_INH: now also U15.2 (QC); no longer U15.15 (QA)
- net BCD_1E0_1: now also RN5.1 (R1.1); no longer RN8.1 (R1.1)
- net BCD_1E0_1_R: now also RN5.8 (R1.2), U12.3 (D4); no longer RN8.8 (R1.2), U13.5 (D6)
- net BCD_1E0_2: now also RN9.3 (R3.1); no longer RN8.2 (R2.1)
- net BCD_1E0_2_R: now also RN9.6 (R3.2), U14.3 (D4); no longer RN8.7 (R2.2), U13.4 (D5)
- net BCD_1E0_4: now also RN5.4 (R4.1); no longer RN8.3 (R3.1)
- net BCD_1E0_4_R: now also RN5.5 (R4.2), U12.4 (D5); no longer RN8.6 (R3.2), U13.3 (D4)
- net BCD_1E0_8: now also RN6.2 (R2.1); no longer RN8.4 (R4.1)
- net BCD_1E0_8_R: now also RN6.7 (R2.2), U12.12 (D1); no longer RN8.5 (R4.2), U13.6 (D7)
- net BCD_1E1_1: now also RN6.3 (R3.1); no longer RN7.1 (R1.1)
- net BCD_1E1_1_R: now also RN6.6 (R3.2), U12.11 (D0); no longer RN7.8 (R1.2), U13.11 (D0)
- net BCD_1E1_2_R: now also U13.5 (D6); no longer U13.13 (D2)
- net BCD_1E1_4: now also RN7.4 (R4.1); no longer RN7.3 (R3.1)
- net BCD_1E1_4_R: now also RN7.5 (R4.2), U13.3 (D4); no longer RN7.6 (R3.2), U13.14 (D3)
- net BCD_1E1_8: now also RN8.2 (R2.1); no longer RN7.4 (R4.1)
- net BCD_1E1_8_R: now also RN8.7 (R2.2); no longer RN7.5 (R4.2)
- net BCD_1E2_1: now also RN3.1 (R1.1); no longer RN4.1 (R1.1)
- net BCD_1E2_1_R: now also RN3.8 (R1.2), U10.3 (D4); no longer RN4.8 (R1.2), U11.5 (D6)
- net BCD_1E2_2: now also RN3.3 (R3.1); no longer RN4.2 (R2.1)
- net BCD_1E2_2_R: now also RN3.6 (R3.2), U10.6 (D7); no longer RN4.7 (R2.2), U11.4 (D5)
- net BCD_1E2_4: now also RN4.1 (R1.1); no longer RN4.3 (R3.1)
- net BCD_1E2_4_R: now also RN4.8 (R1.2), U10.12 (D1); no longer RN4.6 (R3.2), U11.3 (D4)
- net BCD_1E2_8: now also RN4.2 (R2.1); no longer RN4.4 (R4.1)
- net BCD_1E2_8_R: now also RN4.7 (R2.2), U10.11 (D0); no longer RN4.5 (R4.2), U11.6 (D7)
- net BCD_1E3_1: now also RN9.4 (R4.1); no longer RN3.1 (R1.1)
- net BCD_1E3_1_R: now also RN9.5 (R4.2), U14.5 (D6); no longer RN3.8 (R1.2), U11.11 (D0)
- net BCD_1E3_2: now also RN4.4 (R4.1); no longer RN3.2 (R2.1)
- net BCD_1E3_2_R: now also RN4.5 (R4.2), U10.14 (D3); no longer RN3.7 (R2.2), U11.13 (D2)
- net BCD_1E3_4: now also RN2.1 (R1.1); no longer RN3.3 (R3.1)
- net BCD_1E3_4_R: now also RN2.8 (R1.2), U11.13 (D2); no longer RN3.6 (R3.2), U11.14 (D3)
- net BCD_1E3_8: now also RN2.2 (R2.1); no longer RN3.4 (R4.1)
- net BCD_1E3_8_R: now also RN2.7 (R2.2), U11.11 (D0); no longer RN3.5 (R4.2), U11.12 (D1)
- net BCD_1E4_1: now also RN2.4 (R4.1); no longer RN6.1 (R1.1)
- net BCD_1E4_1_R: now also RN2.5 (R4.2), U11.14 (D3); no longer RN6.8 (R1.2), U12.6 (D7)
- net BCD_1E4_2: now also RN5.2 (R2.1); no longer RN6.2 (R2.1)
- net BCD_1E4_2_R: now also RN5.7 (R2.2), U12.5 (D6); no longer RN6.7 (R2.2), U12.3 (D4)
- net BCD_1E4_4: now also RN5.3 (R3.1); no longer RN6.3 (R3.1)
- net BCD_1E4_4_R: now also RN5.6 (R3.2), U12.6 (D7); no longer RN6.6 (R3.2), U12.4 (D5)
- net BCD_1E4_8: now also RN6.1 (R1.1); no longer RN6.4 (R4.1)
- net BCD_1E4_8_R: now also RN6.8 (R1.2), U12.13 (D2); no longer RN6.5 (R4.2), U12.5 (D6)
- net BCD_1E5_1: now also RN9.1 (R1.1); no longer RN5.1 (R1.1)
- net BCD_1E5_1_R: now also RN9.8 (R1.2), U14.6 (D7); no longer RN5.8 (R1.2), U12.11 (D0)
- net BCD_1E5_2: now also RN7.1 (R1.1); no longer RN5.2 (R2.1)
- net BCD_1E5_2_R: now also RN7.8 (R1.2), U13.4 (D5); no longer RN5.7 (R2.2), U12.14 (D3)
- net BCD_1E5_4: now also RN7.3 (R3.1); no longer RN5.3 (R3.1)
- net BCD_1E5_4_R: now also RN7.6 (R3.2), U13.6 (D7); no longer RN5.6 (R3.2), U12.13 (D2)
- net BCD_1E5_8: now also RN8.1 (R1.1); no longer RN5.4 (R4.1)
- net BCD_1E5_8_R: now also RN8.8 (R1.2), U13.13 (D2); no longer RN5.5 (R4.2), U12.12 (D1)
- net BCD_1E6_1: now also RN8.3 (R3.1); no longer RN9.2 (R2.1)
- net BCD_1E6_1_R: now also RN8.6 (R3.2), U13.11 (D0); no longer RN9.7 (R2.2), U14.5 (D6)
- net DATA_CAN_CHANGE: now also RN6.4 (R4.1); no longer RN9.3 (R3.1)
- net DATA_CAN_CHANGE_R: now also RN6.5 (R4.2), U12.14 (D3); no longer RN9.6 (R3.2), U14.11 (D0)
- net FUNC_CMD_42: now also U16.2 (QC); no longer U15.5 (QF)
- net FUNC_CMD_43: now also U16.4 (QE); no longer U15.4 (QE)
- net FUNC_OUT_A: now also RN1.4 (R4.1); no longer RN1.2 (R2.1)
- net FUNC_OUT_A_R: now also RN1.5 (R4.2), U11.3 (D4); no longer RN1.7 (R2.2), U10.13 (D2)
- net FUNC_OUT_B: now also RN1.2 (R2.1); no longer RN1.1 (R1.1)
- net FUNC_OUT_B_R: now also RN1.7 (R2.2), U11.6 (D7); no longer RN1.8 (R1.2), U10.12 (D1)
- net INTEG_2: now also U15.3 (QD); no longer U15.2 (QC)
- net INTEG_4: now also U15.15 (QA); no longer U15.3 (QD)
- net ISO_+5V: now also U14.12 (D1); no longer U14.13 (D2)
- net ISO_GND: now also U14.11 (D0), U14.13 (D2); no longer U14.3 (D4), U14.4 (D5)
- net LED_REMOTE: now also U15.7 (QH); no longer U16.15 (QA)
- net LOCKOUT_N: now also U16.5 (QF); no longer U15.7 (QH)
- net OVERLOAD: now also RN9.2 (R2.1); no longer RN9.4 (R4.1)
- net OVERLOAD_R: now also RN9.7 (R2.2), U14.4 (D5); no longer RN9.5 (R4.2), U14.12 (D1)
- net POL_NEG_R: now also U11.5 (D6); no longer U10.14 (D3)
- net POL_POS: now also RN2.3 (R3.1); no longer RN1.4 (R4.1)
- net POL_POS_R: now also RN2.6 (R3.2), U11.12 (D1); no longer RN1.5 (R4.2), U10.11 (D0)
- net PRINT_LEVEL: now also RN8.4 (R4.1); no longer RN9.1 (R1.1)
- net PRINT_LEVEL_R: now also RN8.5 (R4.2), U13.14 (D3); no longer RN9.8 (R1.2), U14.6 (D7)
- net PRINT_PULSE: now also RN3.2 (R2.1); no longer RN2.1 (R1.1)
- net PRINT_PULSE_R: now also RN3.7 (R2.2), U10.5 (D6); no longer RN2.8 (R1.2), U10.4 (D5)
- net RANGE_CMD_1: now also U15.4 (QE); no longer U16.7 (QH)
- net RANGE_CMD_2: now also U15.5 (QF); no longer U16.5 (QF)
- net RANGE_CMD_4: now also U15.6 (QG); no longer U16.4 (QE)
- net RANGE_OUT_1: now also RN3.4 (R4.1); no longer RN2.2 (R2.1)
- net RANGE_OUT_1_R: now also RN3.5 (R4.2), U10.4 (D5); no longer RN2.7 (R2.2), U10.3 (D4)
- net RANGE_OUT_2: now also RN1.1 (R1.1); no longer RN2.3 (R3.1)
- net RANGE_OUT_2_R: now also RN1.8 (R1.2), U11.4 (D5); no longer RN2.6 (R3.2), U10.5 (D6)
- net RANGE_OUT_4: now also RN4.3 (R3.1); no longer RN2.4 (R4.1)
- net RANGE_OUT_4_R: now also RN4.6 (R3.2), U10.13 (D2); no longer RN2.5 (R4.2), U10.6 (D7)
- net RATIO_N: now also U16.1 (QB); no longer U15.6 (QG)
- net SAMPLE_CONTACT_DRV: now also U16.15 (QA); no longer U16.3 (QD)
- net SAMPLE_PULSE: now also U16.3 (QD); no longer U16.6 (QG)
Other:
- note added: "Isolated serial link (RP2354A SPI0 / PIO): SPI mode 0, MSB first, <= 1 MHz, 40 clocks per transfer. Pulse LATCH low >= 1 us, then clock 5 bytes. LATCH low: the 74HCT165s sample the meter outputs. LATCH rising edge: the 74HC595 outputs take the last two bytes clocked in. /OE (GPIO24) high = command outputs off (the default while the MCU is unpowered or in reset). MISO byte0 U10: 2x10^2 PRINT_PULSE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"
- note removed: "Isolated serial link (RP2354A SPI0 / PIO): SPI mode 0, MSB first, <= 1 MHz, 40 clocks per transfer. Pulse LATCH low >= 1 us, then clock 5 bytes. LATCH low: the 74HCT165s sample the meter outputs. LATCH rising edge: the 74HC595 outputs take the last two bytes clocked in. /OE (GPIO24) high = command outputs off (the default while the MCU is unpowered or in reset). MISO byte0 U10: RANGE_4 RANGE_2 PR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"
