File: atopile/schematic/power_usb.kicad_sch (KiCad schematic)
At the start: 16 parts, among them U19 BF 180, U2 IB0505LS-1WR3, U3 TLV75901PDRVR

Commit message: Run ERC on the schematic; confirm Hi-Z command inputs are inactive
Schematic export:
- Assign real electrical pin types (datasheet-based for the ICs,
  passive otherwise); atopile's EasyEDA symbols type every pin
  input/unspecified, which gave 460 meaningless ERC violations
- Add PWR_FLAGs on the four rails fed through passives (GND, +5V,
  +1V1, VREG_AVDD), write sym/fp library tables and a project file
- Run KiCad ERC as part of the export: 0 errors, 0 warnings
  (negative test: dropping the +5V flag is reported as an error)

Manual section 9, diag 9.2 (70754 board 2): every command input has a
4.7k pull-up to +5V into TTL, contact SAMPLE a 2.2k pull-up, and pulse
SAMPLE is AC-coupled. Hi-Z outputs therefore read as inactive, and the
5.25V HCT high is within TTL ratings. Document this, plus the need to
load PULSE SAMPLE = 0 before enabling the outputs.

Co-Authored-By: Claude Opus 5.5 <noreply@anthropic.com>
Claude-Session: https://claude.ai/code/session_01NqBEt2iCuw3VMJkgzgPtpr
Other:
- note added: "erc_power_flags"
