File: atopile/schematic/dvm.kicad_sch (KiCad schematic)
At the start: 20 parts, among them CN1 DD50P364TXLF, Q1 2N7002, U1 SN74AHCT1G125DBVR, U12 CD74HCT165M96, U13 CD74HCT165M96, U14 CD74HCT165M96, U15 CD74HCT165M96, U16 CD74HCT165M96, U17 74HCT595D,118, U18 74HCT595D,118

Commit message: atopile: pin-swap the shift registers to untangle the DD-50 routing
- scripts/pin_swap.py: treats all 74HCT165 inputs, all 74HCT595 outputs
  and both chain orders as interchangeable, minimises ratsnest length +
  crossings (seeded simulated annealing) and regenerates the pin-map
  block in main.ato and the firmware bit-map tables in README.md
- DVM-side ratsnest: 1544 mm / 839 crossings -> 860 mm / 154 crossings;
  165 chain now follows the physical row (124 mm -> 56 mm)
- place_components.py: fixed register slots (the old centroid sort was
  not idempotent once the DD-50 sat on B.Cu and reversed the row)
- schematic, ERC and fab outputs regenerated; no parts moved

Co-Authored-By: Claude Opus 5.5 <noreply@anthropic.com>
Claude-Session: https://claude.ai/code/session_01NqBEt2iCuw3VMJkgzgPtpr
Connections:
- net +5V_ISO: now also U12.11 (D0), U12.12 (D1); no longer U16.12 (D1), U16.14 (D3)
- net GND_ISO: now also U12.6 (D7), U13.10 (DS), U16.12 (D1); no longer U16.10 (DS), U16.11 (D0), U16.13 (D2)
- net MOSI_ISO: now also U18.14 (DS); no longer U17.14 (DS)
- net SAMPLE_CONTACT_GATE: now also U18.7 (Q7); no longer U17.1 (Q1)
- net SI_CHAIN_1: now also U16.9 (Q7); no longer U13.9 (Q7)
- net SI_CHAIN_2: now also U16.10 (DS); no longer U13.10 (DS)
- net SI_CHAIN_4: now also U13.9 (Q7); no longer U16.9 (Q7)
- net SKB01_D6_1: now also U13.12 (D1); no longer U12.6 (D7)
- net SKB02_D5_8: now also U13.6 (D7); no longer U12.5 (D6)
- net SKB03_D5_4: now also U13.3 (D4); no longer U12.4 (D5)
- net SKB04_D5_2: now also U15.12 (D1); no longer U12.3 (D4)
- net SKB05_D5_1: now also U15.14 (D3); no longer U12.14 (D3)
- net SKB06_D4_8: now also U15.5 (D6); no longer U12.13 (D2)
- net SKB07_D4_4: now also U15.3 (D4); no longer U12.12 (D1)
- net SKB08_D4_2: now also U14.13 (D2); no longer U12.11 (D0)
- net SKB09_D4_1: now also U14.6 (D7); no longer U13.6 (D7)
- net SKB10_D3_8: now also U14.4 (D5); no longer U13.5 (D6)
- net SKB11_D3_4: now also U16.11 (D0); no longer U13.4 (D5)
- net SKB12_D3_2: now also U16.14 (D3); no longer U13.3 (D4)
- net SKB13_D3_1: now also U16.5 (D6); no longer U13.14 (D3)
- net SKB14_D2_8: now also U16.3 (D4); no longer U13.13 (D2)
- net SKB15_D2_4: now also U12.14 (D3); no longer U13.12 (D1)
- net SKB16_D2_2: now also U12.4 (D5); no longer U13.11 (D0)
- net SKB17_D2_1: now also U12.3 (D4); no longer U14.6 (D7)
- net SKB18_D1_8: now also U13.14 (D3); no longer U14.5 (D6)
- net SKB19_D1_4: now also U13.5 (D6); no longer U14.4 (D5)
- net SKB20_D1_2: now also U15.11 (D0); no longer U14.3 (D4)
- net SKB21_D1_1: now also U15.13 (D2); no longer U14.14 (D3)
- net SKB22_D0_8: now also U15.6 (D7); no longer U14.13 (D2)
- net SKB23_D0_4: now also U15.4 (D5); no longer U14.12 (D1)
- net SKB25_D0_1: now also U14.12 (D1); no longer U15.6 (D7)
- net SKB26_POL_POS: now also U14.14 (D3); no longer U15.5 (D6)
- net SKB27_POL_NEG: now also U14.5 (D6); no longer U15.4 (D5)
- net SKB28_FUNC_OUT_A: now also U14.3 (D4); no longer U15.3 (D4)
- net SKB29_FUNC_OUT_B: now also U16.13 (D2); no longer U15.14 (D3)
- net SKB30_RANGE_OUT_4: now also U16.6 (D7); no longer U15.13 (D2)
- net SKB31_RANGE_OUT_2: now also U16.4 (D5); no longer U15.12 (D1)
- net SKB32_RANGE_OUT_1: now also U12.13 (D2); no longer U15.11 (D0)
- net SKB33_PRINT_PULSE: now also U12.5 (D6); no longer U16.6 (D7)
- net SKB34_PRINT_LEVEL: now also U13.11 (D0); no longer U16.5 (D6)
- net SKB35_DATA_CAN_CHANGE: now also U13.13 (D2); no longer U16.4 (D5)
- net SKB36_OVERLOAD: now also U13.4 (D5); no longer U16.3 (D4)
- net SKB38_LOCKOUT: now also U18.1 (Q1); no longer U17.15 (Q0)
- net SKB40_SAMPLE_PULSE: now also U18.4 (Q4); no longer U17.2 (Q2)
- net SKB41_RATIO: now also U18.5 (Q5); no longer U17.3 (Q3)
- net SKB42_FUNC_CMD_A: now also U18.6 (Q6); no longer U17.4 (Q4)
- net SKB43_FUNC_CMD_B: now also U17.15 (Q0); no longer U17.5 (Q5)
- net SKB44_INT_TIME_4: now also U17.1 (Q1); no longer U17.6 (Q6)
- net SKB45_INT_TIME_2: now also U17.2 (Q2); no longer U17.7 (Q7)
- net SKB46_INT_TIME_1: now also U17.3 (Q3); no longer U18.15 (Q0)
- net SKB47_AUTORANGE: now also U17.4 (Q4); no longer U18.1 (Q1)
- net SKB48_RANGE_CMD_1: now also U17.5 (Q5); no longer U18.2 (Q2)
- net SKB49_RANGE_CMD_2: now also U17.6 (Q6); no longer U18.3 (Q3)
- net SKB50_RANGE_CMD_4: now also U17.7 (Q7); no longer U18.4 (Q4)
- net SO_CHAIN_1: now also U17.14 (DS), U18.9 (Q7S); no longer U17.9 (Q7S), U18.14 (DS)
Other:
- moved on the sheet: C1, C30, C31, C32, C34, C36, R10, U1, U12, U13, U14, U15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

Commit message: atopile: move DVM-side parts for routing, then redo the pin swap
- optimise_placement.py result: IC row (E->W) 165,595,165,595,165,165,165
  with the 165s turned 180 deg; DRDY buffer to the west end next to SKB 34;
  SAMPLE MOSFET + pull-down south of the DD-50 in line with SKB 39; opto
  order W->E DRDY, MISO, LATCH, MOSI, OE_N, SCK
- pin_swap.py: control nets (SCK/LATCH/OE_N/DRDY, SKB 39 drain, MCU<->opto)
  now count for crossings; longer annealing and a chain-reversal move so
  all restarts converge
- DVM ratsnest incl. control nets: 1206 mm / 297 crossings (pin swap only)
  -> 985 mm / 112 crossings (original: 1889 mm / 1000)
- schematic, ERC, fab outputs, placement picture and README regenerated

Co-Authored-By: Claude Opus 5.5 <noreply@anthropic.com>
Claude-Session: https://claude.ai/code/session_01NqBEt2iCuw3VMJkgzgPtpr
Connections:
- net +5V_ISO: now also U14.14 (D3), U16.13 (D2); no longer U12.11 (D0), U12.12 (D1)
- net GND_ISO: now also U12.10 (DS), U16.14 (D3); no longer U12.6 (D7), U13.10 (DS)
- net MISO_ISO: now also U16.9 (Q7); no longer U12.9 (Q7)
- net SAMPLE_CONTACT_GATE: now also U18.1 (Q1); no longer U18.7 (Q7)
- net SI_CHAIN_1: now also U15.9 (Q7), U16.10 (DS); no longer U12.10 (DS), U16.9 (Q7)
- net SI_CHAIN_2: now also U15.10 (DS); no longer U16.10 (DS)
- net SI_CHAIN_3: now also U13.9 (Q7); no longer U15.9 (Q7)
- net SI_CHAIN_4: now also U12.9 (Q7), U13.10 (DS); no longer U13.9 (Q7), U15.10 (DS)
- net SKB01_D6_1: now also U16.6 (D7); no longer U13.12 (D1)
- net SKB02_D5_8: now also U16.4 (D5); no longer U13.6 (D7)
- net SKB03_D5_4: now also U15.5 (D6); no longer U13.3 (D4)
- net SKB04_D5_2: now also U15.11 (D0); no longer U15.12 (D1)
- net SKB05_D5_1: now also U15.13 (D2); no longer U15.14 (D3)
- net SKB06_D4_8: now also U14.6 (D7); no longer U15.5 (D6)
- net SKB07_D4_4: now also U14.4 (D5); no longer U15.3 (D4)
- net SKB08_D4_2: now also U14.11 (D0); no longer U14.13 (D2)
- net SKB09_D4_1: now also U14.13 (D2); no longer U14.6 (D7)
- net SKB10_D3_8: now also U13.4 (D5); no longer U14.4 (D5)
- net SKB11_D3_4: now also U13.6 (D7); no longer U16.11 (D0)
- net SKB12_D3_2: now also U13.13 (D2); no longer U16.14 (D3)
- net SKB13_D3_1: now also U13.11 (D0); no longer U16.5 (D6)
- net SKB14_D2_8: now also U12.5 (D6); no longer U16.3 (D4)
- net SKB16_D2_2: now also U12.12 (D1); no longer U12.4 (D5)
- net SKB17_D2_1: now also U12.11 (D0); no longer U12.3 (D4)
- net SKB18_D1_8: now also U16.3 (D4); no longer U13.14 (D3)
- net SKB19_D1_4: now also U15.6 (D7); no longer U13.5 (D6)
- net SKB20_D1_2: now also U15.3 (D4); no longer U15.11 (D0)
- net SKB21_D1_1: now also U15.12 (D1); no longer U15.13 (D2)
- net SKB22_D0_8: now also U15.14 (D3); no longer U15.6 (D7)
- net SKB23_D0_4: now also U14.5 (D6); no longer U15.4 (D5)
- net SKB24_D0_2: now also U14.3 (D4); no longer U14.11 (D0)
- net SKB26_POL_POS: now also U13.3 (D4); no longer U14.14 (D3)
- net SKB27_POL_NEG: now also U13.5 (D6); no longer U14.5 (D6)
- net SKB28_FUNC_OUT_A: now also U13.14 (D3); no longer U14.3 (D4)
- net SKB29_FUNC_OUT_B: now also U13.12 (D1); no longer U16.13 (D2)
- net SKB30_RANGE_OUT_4: now also U12.3 (D4); no longer U16.6 (D7)
- net SKB31_RANGE_OUT_2: now also U12.4 (D5); no longer U16.4 (D5)
- net SKB32_RANGE_OUT_1: now also U12.6 (D7); no longer U12.13 (D2)
- net SKB33_PRINT_PULSE: now also U12.13 (D2); no longer U12.5 (D6)
- net SKB34_PRINT_LEVEL: now also U16.5 (D6); no longer U13.11 (D0)
- net SKB35_DATA_CAN_CHANGE: now also U16.11 (D0); no longer U13.13 (D2)
- net SKB36_OVERLOAD: now also U15.4 (D5); no longer U13.4 (D5)
- net SKB38_LOCKOUT: now also U18.15 (Q0); no longer U18.1 (Q1)
- net SKB40_SAMPLE_PULSE: now also U18.6 (Q6); no longer U18.4 (Q4)
- net SKB42_FUNC_CMD_A: now also U18.3 (Q3); no longer U18.6 (Q6)
- net SKB43_FUNC_CMD_B: now also U18.2 (Q2); no longer U17.15 (Q0)
- net SKB44_INT_TIME_4: now also U18.4 (Q4); no longer U17.1 (Q1)
- net SKB45_INT_TIME_2: now also U17.15 (Q0); no longer U17.2 (Q2)
- net SKB46_INT_TIME_1: now also U17.5 (Q5); no longer U17.3 (Q3)
- net SKB48_RANGE_CMD_1: now also U17.3 (Q3); no longer U17.5 (Q5)
- net SKB49_RANGE_CMD_2: now also U17.1 (Q1); no longer U17.6 (Q6)
- net SKB50_RANGE_CMD_4: now also U17.2 (Q2); no longer U17.7 (Q7)
Other:
- moved on the sheet: C1, C30, C31, C32, C34, R10, U1, U12, U13, U14, U15, U16
