File: konnect/solartron_7075_interface_konnect.kicad_sch (KiCad schematic)
At the start: 93 parts, among them J1 DD-50 Male (Solartron SKB), J2 USB_B, J3 SWD, Q1 2N7002, SW1 BOOTSEL, SW2 RUN, U1 RP2354A, U11 AMS1117-3.3, U12 SN74LVC165APWR, U13 SN74LVC165APWR, U14 SN74LVC165APWR, U15 SN74LVC165APWR, U16 SN74LVC165APWR, U17 74LVC595APW, U18 74LVC595APW, U19 74LVC1G17, U2 USBLC6-2SC6, U3 AP2112K-3.3, U4 TLP2361, U5 TLP2361, U6 TLP2361, U7 TLP2361, U8 TLP2361, U9 TLP2361, Y1 12MHz

Commit message: Konnect: Solartron 7075 interface - PCB placed, routed and poured
- 74 x 74 mm 2-layer board. DD-50 (J1) on the bottom face to plug into the
  meter's SKB socket and fix the board by its jackscrews; vertical USB-B (J2)
  on the top face.
- Meter side (GND_ISO): '595 command outputs above the D-sub pin field, 100k
  pull-down networks and the five-'165 input chain below it, AMS1117 iso LDO.
- Six TLP2361 optos and the B0505S module straddle a ~4.8 mm copper-free
  isolation band; no net crosses the barrier.
- USB side (GND): RP2354A, AP2112K, USBLC6, BOOTSEL/RUN, SWD header.
- Signals autorouted with Freerouting via Konnect (band and edge keepouts);
  GND / GND_ISO poured on both layers with stitching vias and bridge tracks.
- DRC: 0 unconnected items; 1 cosmetic starved-thermal on C17 pad 2
  (connected by track); remaining items are warnings.
- fab/: Gerbers + drill, JLCPCB BOM with LCSC numbers, position file, PDFs.

Co-Authored-By: Claude Opus 5.5 <noreply@anthropic.com>
Parts:
- U1: footprint solartron:QFN-60-1EP_7x7mm_P0.4mm_EP3.4x3.4mm_RectPads -> Package_DFN_QFN:QFN-60-1EP_7x7mm_P0.4mm_EP3.4x3.4mm
Changed lines of the file:
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@@
 			)
 		)
-		(property "Footprint" "solartron:QFN-60-1EP_7x7mm_P0.4mm_EP3.4x3.4mm_RectPads"
+		(property "Footprint" "Package_DFN_QFN:QFN-60-1EP_7x7mm_P0.4mm_EP3.4x3.4mm"
 			(at 106.68 193.04 0)
 			(hide yes)

Commit message: Konnect: pin-swap the shift registers and resistor arrays, re-route meter side
- Re-assigned the 36 DVM inputs across the five '165s and nine 100k arrays,
  within and between identical parts, so each array feeds one side of one
  '165 in D-sub pin order. Reordered the '595 outputs to match the D-sub
  top row. U16 keeps its 0,0,1,1 signature; the schematic note now carries
  the full MISO/MOSI bit map (SAMPLE moved to U18 QA/QC).
- Pre-placed the '165 LOAD/SCK escapes and bottom-layer buses, and ground
  pockets for the arrays and the '165 GND/CLK INH pins, then re-routed the
  meter side with Freerouting. The USB side is unchanged.
- Meter-side signals: 2,374 mm / 111 vias -> 1,692 mm / 55 vias; the 36
  input nets alone: 1,343 mm / 53 vias -> 781 mm / 7 vias.
- ERC clean. DRC: 0 unconnected, 4 cosmetic starved-thermal errors
  (C17, C24, C30, C31). Fab outputs regenerated; BOM and positions unchanged.

Co-Authored-By: Claude Opus 5.5 <noreply@anthropic.com>
Connections:
- net BCD0_1: now also RN7.3 (R3.1), U16.4 (D5); no longer RN7.1 (R1.1), U16.3 (D4)
- net BCD0_2: now also RN7.1 (R1.1), U16.6 (D7); no longer RN6.4 (R4.1), U16.4 (D5)
- net BCD0_4: now also U12.12 (D1); no longer U16.5 (D6)
- net BCD0_8: now also RN6.1 (R1.1), U12.14 (D3); no longer RN6.2 (R2.1), U16.6 (D7)
- net BCD1_1: now also RN9.3 (R3.1), U12.4 (D5); no longer RN6.1 (R1.1), U15.11 (D0)
- net BCD1_2: now also RN9.1 (R1.1), U12.6 (D7); no longer RN5.4 (R4.1), U15.12 (D1)
- net BCD1_4: now also RN1.2 (R2.1), U13.13 (D2); no longer RN5.3 (R3.1), U15.13 (D2)
- net BCD1_8: now also RN8.3 (R3.1), U13.4 (D5); no longer RN5.2 (R2.1), U15.14 (D3)
- net BCD2_1: now also RN5.4 (R4.1), U15.11 (D0); no longer RN5.1 (R1.1), U15.3 (D4)
- net BCD2_2: now also RN5.2 (R2.1), U15.13 (D2); no longer RN4.4 (R4.1), U15.4 (D5)
- net BCD2_4: now also RN4.4 (R4.1), U15.3 (D4); no longer RN4.3 (R3.1), U15.5 (D6)
- net BCD2_8: now also U15.5 (D6); no longer U15.6 (D7)
- net BCD3_1: now also RN3.4 (R4.1); no longer RN4.1 (R1.1)
- net BCD3_2: now also RN3.2 (R2.1), U14.13 (D2); no longer RN3.4 (R4.1), U14.12 (D1)
- net BCD3_4: now also RN2.4 (R4.1), U14.3 (D4); no longer RN3.3 (R3.1), U14.13 (D2)
- net BCD3_8: now also RN2.2 (R2.1), U14.5 (D6); no longer RN3.2 (R2.1), U14.14 (D3)
- net BCD4_1: now also RN7.4 (R4.1), U16.3 (D4); no longer RN3.1 (R1.1), U14.3 (D4)
- net BCD4_2: now also RN7.2 (R2.1), U16.5 (D6); no longer RN2.4 (R4.1), U14.4 (D5)
- net BCD4_4: now also RN6.4 (R4.1), U12.11 (D0); no longer RN2.3 (R3.1), U14.5 (D6)
- net BCD4_8: now also RN6.2 (R2.1), U12.13 (D2); no longer RN2.2 (R2.1), U14.6 (D7)
- net BCD5_1: now also RN9.4 (R4.1), U12.3 (D4); no longer RN2.1 (R1.1), U13.11 (D0)
- net BCD5_2: now also RN9.2 (R2.1), U12.5 (D6); no longer RN1.4 (R4.1), U13.12 (D1)
- net BCD5_4: now also RN1.4 (R4.1), U13.11 (D0); no longer RN1.3 (R3.1), U13.13 (D2)
- net BCD5_8: now also RN1.1 (R1.1); no longer RN1.2 (R2.1)
- net BCD6_1: now also RN8.2 (R2.1), U13.5 (D6); no longer RN1.1 (R1.1), U13.3 (D4)
- net CMD_AUTORANGE_INH: now also U17.4 (QE); no longer U17.3 (QD)
- net CMD_FN_42: now also U18.3 (QD); no longer U18.15 (QA)
- net CMD_FN_43: now also U18.4 (QE); no longer U18.1 (QB)
- net CMD_FPL_N: now also U18.1 (QB); no longer U18.2 (QC)
- net CMD_INT_1: now also U17.3 (QD); no longer U17.4 (QE)
- net CMD_INT_2: now also U17.2 (QC); no longer U17.5 (QF)
- net CMD_INT_4: now also U17.1 (QB); no longer U17.6 (QG)
- net CMD_RATIO_N: now also U17.15 (QA); no longer U17.7 (QH)
- net CMD_RNG_1: now also U17.5 (QF); no longer U17.15 (QA)
- net CMD_RNG_2: now also U17.6 (QG); no longer U17.1 (QB)
- net CMD_RNG_4: now also U17.7 (QH); no longer U17.2 (QC)
- net CMD_SAMPLE_PULSE: now also U18.2 (QC); no longer U18.3 (QD)
- net DATA_CAN_CHANGE: now also RN8.4 (R4.1), U13.3 (D4); no longer RN9.3 (R3.1), U12.5 (D6)
- net FN_OUT_28: now also RN3.1 (R1.1), U14.14 (D3); no longer RN7.4 (R4.1), U12.12 (D1)
- net FN_OUT_29: now also RN3.3 (R3.1), U14.12 (D1); no longer RN8.1 (R1.1), U12.11 (D0)
- net OVERLOAD: now also RN1.3 (R3.1), U13.12 (D1); no longer RN9.4 (R4.1), U12.4 (D5)
- net POL_NEG: now also RN2.3 (R3.1), U14.4 (D5); no longer RN7.3 (R3.1), U12.13 (D2)
- net POL_POS: now also RN2.1 (R1.1), U14.6 (D7); no longer RN7.2 (R2.1), U12.14 (D3)
- net PRINT_LEVEL: now also RN8.1 (R1.1), U13.6 (D7); no longer RN9.2 (R2.1), U12.6 (D7)
- net PRINT_PULSE: now also RN5.3 (R3.1), U15.12 (D1); no longer RN9.1 (R1.1), U12.3 (D4)
- net RNG_OUT_1: now also RN5.1 (R1.1), U15.14 (D3); no longer RN8.4 (R4.1), U13.4 (D5)
- net RNG_OUT_2: now also RN4.3 (R3.1), U15.4 (D5); no longer RN8.3 (R3.1), U13.5 (D6)
- net RNG_OUT_4: now also RN4.1 (R1.1), U15.6 (D7); no longer RN8.2 (R2.1), U13.6 (D7)
- net SAMPLE_CONTACT_DRV: now also U18.15 (QA); no longer U18.4 (QE)

Commit message: Konnect: move the meter-side parts and lay out the input wiring by script
- U16 (four DVM inputs) moves to the right-hand end so the nine used '165
  input sides sit in a row at twice the D-sub group pitch; each array sits
  under its four D-sub pins, turned to face the connector. The 36 input
  tracks follow one repeated pattern: straight into the array, out between
  its pad rows, and into each '165 side from outside and from under the
  body. One via (DD-50 pin 36, which sits above pin 3).
- '165 decoupling caps moved onto the chips with a bottom-layer +3V3_ISO
  spine; C29 moved above the regulator; U19 turned to face U13.
- Both shift-register chains now run in board order (MOSI -> U18 -> U17 ->
  U16 -> U15 -> U14 -> U12 -> U13 -> MISO) and CMD_RATIO_N moves to U18 QD.
  The schematic note carries the new bit map.
- Control buses, supply rails, SIPO links and the '165 chain were also laid
  by script; Freerouting did the rest. USB side unchanged.
- Meter-side signals: 1,692 mm / 55 vias -> 1,558 mm / 36 vias; the 36
  input nets: 781 mm / 7 vias -> 655 mm / 1 via.
- ERC clean. DRC: 0 unconnected, one cosmetic starved thermal (C17, as in
  the first layout). Fab outputs and positions regenerated; BOM unchanged.

Co-Authored-By: Claude Opus 5.5 <noreply@anthropic.com>
Connections:
- net BCD0_1: now also RN7.2 (R2.1), U14.5 (D6); no longer RN7.3 (R3.1), U16.4 (D5)
- net BCD0_2: now also RN7.4 (R4.1), U14.4 (D5); no longer RN7.1 (R1.1), U16.6 (D7)
- net BCD0_4: now also RN6.2 (R2.1), U12.14 (D3); no longer RN6.3 (R3.1), U12.12 (D1)
- net BCD0_8: now also RN6.4 (R4.1), U12.11 (D0); no longer RN6.1 (R1.1), U12.14 (D3)
- net BCD1_1: now also RN9.2 (R2.1), U12.5 (D6); no longer RN9.3 (R3.1), U12.4 (D5)
- net BCD1_2: now also RN9.4 (R4.1), U12.4 (D5); no longer RN9.1 (R1.1), U12.6 (D7)
- net BCD1_4: now also RN1.3 (R3.1), U13.12 (D1); no longer RN1.2 (R2.1), U13.13 (D2)
- net BCD1_8: now also U13.3 (D4); no longer U13.4 (D5)
- net BCD2_1: now also RN5.1 (R1.1), U16.6 (D7); no longer RN5.4 (R4.1), U15.11 (D0)
- net BCD2_2: now also RN5.3 (R3.1), U16.3 (D4); no longer RN5.2 (R2.1), U15.13 (D2)
- net BCD2_4: now also RN4.1 (R1.1), U15.13 (D2); no longer RN4.4 (R4.1), U15.3 (D4)
- net BCD2_8: now also RN4.3 (R3.1), U15.12 (D1); no longer RN4.2 (R2.1), U15.5 (D6)
- net BCD3_1: now also RN3.1 (R1.1), U15.6 (D7); no longer RN3.4 (R4.1), U14.11 (D0)
- net BCD3_2: now also RN3.3 (R3.1), U15.3 (D4); no longer RN3.2 (R2.1), U14.13 (D2)
- net BCD3_4: now also RN2.1 (R1.1), U14.13 (D2); no longer RN2.4 (R4.1), U14.3 (D4)
- net BCD3_8: now also RN2.3 (R3.1), U14.12 (D1); no longer RN2.2 (R2.1), U14.5 (D6)
- net BCD4_1: now also RN7.1 (R1.1), U14.6 (D7); no longer RN7.4 (R4.1), U16.3 (D4)
- net BCD4_2: now also RN7.3 (R3.1), U14.3 (D4); no longer RN7.2 (R2.1), U16.5 (D6)
- net BCD4_4: now also RN6.1 (R1.1), U12.13 (D2); no longer RN6.4 (R4.1), U12.11 (D0)
- net BCD4_8: now also RN6.3 (R3.1), U12.12 (D1); no longer RN6.2 (R2.1), U12.13 (D2)
- net BCD5_1: now also RN9.1 (R1.1), U12.6 (D7); no longer RN9.4 (R4.1), U12.3 (D4)
- net BCD5_2: now also RN9.3 (R3.1), U12.3 (D4); no longer RN9.2 (R2.1), U12.5 (D6)
- net BCD5_4: now also RN1.1 (R1.1), U13.13 (D2); no longer RN1.4 (R4.1), U13.11 (D0)
- net BCD5_8: now also RN1.4 (R4.1), U13.11 (D0); no longer RN1.1 (R1.1), U13.14 (D3)
- net BCD6_1: now also RN8.1 (R1.1), U13.6 (D7); no longer RN8.2 (R2.1), U13.5 (D6)
- net CMD_FN_42: now also U18.4 (QE); no longer U18.3 (QD)
- net CMD_FN_43: now also U18.5 (QF); no longer U18.4 (QE)
- net CMD_RATIO_N: now also U18.3 (QD); no longer U17.15 (QA)
- net DATA_CAN_CHANGE: now also RN8.2 (R2.1), U13.5 (D6); no longer RN8.4 (R4.1), U13.3 (D4)
- net FN_OUT_28: now also RN3.4 (R4.1), U15.4 (D5); no longer RN3.1 (R1.1), U14.14 (D3)
- net FN_OUT_29: now also RN3.2 (R2.1), U15.5 (D6); no longer RN3.3 (R3.1), U14.12 (D1)
- net ISO_MISO: now also U13.9 (Q7); no longer U12.9 (Q7)
- net ISO_MOSI: now also U18.14 (SER); no longer U17.14 (SER)
- net OVERLOAD: now also RN1.2 (R2.1), U13.14 (D3); no longer RN1.3 (R3.1), U13.12 (D1)
- net PISO_CH1: now also U12.9 (Q7), U13.10 (DS); no longer U12.10 (DS), U13.9 (Q7)
- net PISO_CH2: now also U12.10 (DS); no longer U13.10 (DS)
- net POL_NEG: now also RN2.2 (R2.1), U14.14 (D3); no longer RN2.3 (R3.1), U14.4 (D5)
- net POL_POS: now also RN2.4 (R4.1), U14.11 (D0); no longer RN2.1 (R1.1), U14.6 (D7)
- net PRINT_LEVEL: now also RN8.4 (R4.1), U13.4 (D5); no longer RN8.1 (R1.1), U13.6 (D7)
- net PRINT_PULSE: now also RN5.2 (R2.1), U16.5 (D6); no longer RN5.3 (R3.1), U15.12 (D1)
- net RNG_OUT_1: now also RN5.4 (R4.1), U16.4 (D5); no longer RN5.1 (R1.1), U15.14 (D3)
- net RNG_OUT_2: now also RN4.2 (R2.1), U15.14 (D3); no longer RN4.3 (R3.1), U15.4 (D5)
- net RNG_OUT_4: now also RN4.4 (R4.1), U15.11 (D0); no longer RN4.1 (R1.1), U15.6 (D7)
- net SIPO_CH1: now also U17.14 (SER), U18.9 (QH'); no longer U17.9 (QH'), U18.14 (SER)
- net SIPO_LOOP: now also U17.9 (QH'); no longer U18.9 (QH')
