File: skidl/output/solartron_7075_interface_unplaced.kicad_pcb (KiCad board)
At the start: 2 copper layers, 94 parts, among them J1 DD-50 plug, J2 USB_B, J3 SWD, Q1 2N7002, SW1 BOOTSEL, SW2 RESET, U1 RP2354A, U10 74HCT165, U11 74HCT165, U12 74HCT165, U13 74HCT165, U14 74HCT165, U15 74HC595, U16 74HC595, U2 AP2112K-3.3, U3 USBLC6-2SC6, U4 78L05, U5 TLP2361, U6 TLP2361, U7 TLP2361, U8 TLP2361, U9 TLP2361, Y1 12MHz

Commit message: skidl: tidy meter-side routing by pin swapping within parts
Reassign the D inputs of the 74HCT165s (U14's link-check inputs included),
the channels of the resistor arrays and the outputs of the 74HC595s, found by
scripts/optimise_pins.py (simulated annealing on straight-line crossings and
length; no part moved, no signal moved to another part). Re-routed with
Freerouting:

  arrays -> 74HCT165s: 64 -> 0 crossings, 441 -> 351 mm of track
  74HC595s -> J1:      36 -> 8 crossings, 265 -> 205 mm
  J1 -> arrays:       148 -> 102 crossings, 513 -> 481 mm
  whole board:        2428 -> 2227 mm of track, 262 -> 260 vias

DRC, ERC and schematic parity remain clean. The bit maps in the README and
the schematic notes (now generated from the netlist) follow the new
assignment; the link-check pattern is now 0011 on U14 D5..D2.

Co-Authored-By: Claude Opus 5.5 <noreply@anthropic.com>
Claude-Session: https://claude.ai/code/session_01ERGgANCwEg9niX4WLDjBj2
Connections:
- RN1 pad 1: POL_POS -> FUNC_OUT_B
- RN1 pad 2: POL_NEG -> FUNC_OUT_A
- RN1 pad 3: FUNC_OUT_A -> POL_NEG
- RN1 pad 4: FUNC_OUT_B -> POL_POS
- RN1 pad 5: FUNC_OUT_B_R -> POL_POS_R
- RN1 pad 6: FUNC_OUT_A_R -> POL_NEG_R
- RN1 pad 7: POL_NEG_R -> FUNC_OUT_A_R
- RN1 pad 8: POL_POS_R -> FUNC_OUT_B_R
- RN2 pad 1: RANGE_OUT_4 -> PRINT_PULSE
- RN2 pad 2: RANGE_OUT_2 -> RANGE_OUT_1
- RN2 pad 3: RANGE_OUT_1 -> RANGE_OUT_2
- RN2 pad 4: PRINT_PULSE -> RANGE_OUT_4
- RN2 pad 5: PRINT_PULSE_R -> RANGE_OUT_4_R
- RN2 pad 6: RANGE_OUT_1_R -> RANGE_OUT_2_R
- RN2 pad 7: RANGE_OUT_2_R -> RANGE_OUT_1_R
- RN2 pad 8: RANGE_OUT_4_R -> PRINT_PULSE_R
- RN3 pad 1: BCD_1E3_8 -> BCD_1E3_1
- RN3 pad 2: BCD_1E3_4 -> BCD_1E3_2
- RN3 pad 3: BCD_1E3_2 -> BCD_1E3_4
- RN3 pad 4: BCD_1E3_1 -> BCD_1E3_8
- RN3 pad 5: BCD_1E3_1_R -> BCD_1E3_8_R
- RN3 pad 6: BCD_1E3_2_R -> BCD_1E3_4_R
- RN3 pad 7: BCD_1E3_4_R -> BCD_1E3_2_R
- RN3 pad 8: BCD_1E3_8_R -> BCD_1E3_1_R
- RN4 pad 1: BCD_1E2_8 -> BCD_1E2_1
- RN4 pad 2: BCD_1E2_4 -> BCD_1E2_2
- RN4 pad 3: BCD_1E2_2 -> BCD_1E2_4
- RN4 pad 4: BCD_1E2_1 -> BCD_1E2_8
- RN4 pad 5: BCD_1E2_1_R -> BCD_1E2_8_R
- RN4 pad 6: BCD_1E2_2_R -> BCD_1E2_4_R
- RN4 pad 7: BCD_1E2_4_R -> BCD_1E2_2_R
- RN4 pad 8: BCD_1E2_8_R -> BCD_1E2_1_R
- RN5 pad 1: BCD_1E5_8 -> BCD_1E5_1
- RN5 pad 2: BCD_1E5_4 -> BCD_1E5_2
- RN5 pad 3: BCD_1E5_2 -> BCD_1E5_4
- RN5 pad 4: BCD_1E5_1 -> BCD_1E5_8
- RN5 pad 5: BCD_1E5_1_R -> BCD_1E5_8_R
- RN5 pad 6: BCD_1E5_2_R -> BCD_1E5_4_R
- RN5 pad 7: BCD_1E5_4_R -> BCD_1E5_2_R
- RN5 pad 8: BCD_1E5_8_R -> BCD_1E5_1_R
- RN6 pad 1: BCD_1E4_8 -> BCD_1E4_1
- RN6 pad 2: BCD_1E4_4 -> BCD_1E4_2
- RN6 pad 3: BCD_1E4_2 -> BCD_1E4_4
- RN6 pad 4: BCD_1E4_1 -> BCD_1E4_8
- RN6 pad 5: BCD_1E4_1_R -> BCD_1E4_8_R
- RN6 pad 6: BCD_1E4_2_R -> BCD_1E4_4_R
- RN6 pad 7: BCD_1E4_4_R -> BCD_1E4_2_R
- RN6 pad 8: BCD_1E4_8_R -> BCD_1E4_1_R
- RN7 pad 1: BCD_1E1_8 -> BCD_1E1_1
- RN7 pad 2: BCD_1E1_4 -> BCD_1E1_2
- RN7 pad 3: BCD_1E1_2 -> BCD_1E1_4
- RN7 pad 4: BCD_1E1_1 -> BCD_1E1_8
- RN7 pad 5: BCD_1E1_1_R -> BCD_1E1_8_R
- RN7 pad 6: BCD_1E1_2_R -> BCD_1E1_4_R
- RN7 pad 7: BCD_1E1_4_R -> BCD_1E1_2_R
- RN7 pad 8: BCD_1E1_8_R -> BCD_1E1_1_R
- RN8 pad 1: BCD_1E0_8 -> BCD_1E0_1
- RN8 pad 2: BCD_1E0_4 -> BCD_1E0_2
- RN8 pad 3: BCD_1E0_2 -> BCD_1E0_4
- RN8 pad 4: BCD_1E0_1 -> BCD_1E0_8
- RN8 pad 5: BCD_1E0_1_R -> BCD_1E0_8_R
- RN8 pad 6: BCD_1E0_2_R -> BCD_1E0_4_R
- RN8 pad 7: BCD_1E0_4_R -> BCD_1E0_2_R
- RN8 pad 8: BCD_1E0_8_R -> BCD_1E0_1_R
- RN9 pad 2: DATA_CAN_CHANGE -> BCD_1E6_1
- RN9 pad 3: OVERLOAD -> DATA_CAN_CHANGE
- RN9 pad 4: BCD_1E6_1 -> OVERLOAD
- RN9 pad 5: BCD_1E6_1_R -> OVERLOAD_R
- RN9 pad 6: OVERLOAD_R -> DATA_CAN_CHANGE_R
- RN9 pad 7: DATA_CAN_CHANGE_R -> BCD_1E6_1_R
- U10 pad 11: PRINT_PULSE_R -> POL_POS_R
- U10 pad 12: RANGE_OUT_1_R -> FUNC_OUT_B_R
- U10 pad 13: RANGE_OUT_2_R -> FUNC_OUT_A_R
- U10 pad 14: RANGE_OUT_4_R -> POL_NEG_R
- U10 pad 3: FUNC_OUT_B_R -> RANGE_OUT_1_R
- U10 pad 4: FUNC_OUT_A_R -> PRINT_PULSE_R
- U10 pad 5: POL_NEG_R -> RANGE_OUT_2_R
- U10 pad 6: POL_POS_R -> RANGE_OUT_4_R
- U11 pad 11: BCD_1E2_1_R -> BCD_1E3_1_R
- U11 pad 12: BCD_1E2_2_R -> BCD_1E3_8_R
- U11 pad 13: BCD_1E2_4_R -> BCD_1E3_2_R
- U11 pad 14: BCD_1E2_8_R -> BCD_1E3_4_R
- U11 pad 3: BCD_1E3_1_R -> BCD_1E2_4_R
- U11 pad 4: BCD_1E3_2_R -> BCD_1E2_2_R
- U11 pad 5: BCD_1E3_4_R -> BCD_1E2_1_R
- U11 pad 6: BCD_1E3_8_R -> BCD_1E2_8_R
- U12 pad 11: BCD_1E4_1_R -> BCD_1E5_1_R
- U12 pad 12: BCD_1E4_2_R -> BCD_1E5_8_R
- U12 pad 13: BCD_1E4_4_R -> BCD_1E5_4_R
- U12 pad 14: BCD_1E4_8_R -> BCD_1E5_2_R
- U12 pad 3: BCD_1E5_1_R -> BCD_1E4_2_R
- U12 pad 4: BCD_1E5_2_R -> BCD_1E4_4_R
- U12 pad 5: BCD_1E5_4_R -> BCD_1E4_8_R
- U12 pad 6: BCD_1E5_8_R -> BCD_1E4_1_R
- U13 pad 11: BCD_1E0_1_R -> BCD_1E1_1_R
- U13 pad 12: BCD_1E0_2_R -> BCD_1E1_8_R
- U13 pad 13: BCD_1E0_4_R -> BCD_1E1_2_R
- U13 pad 14: BCD_1E0_8_R -> BCD_1E1_4_R
- U13 pad 3: BCD_1E1_1_R -> BCD_1E0_4_R
- U13 pad 4: BCD_1E1_2_R -> BCD_1E0_2_R
- U13 pad 5: BCD_1E1_4_R -> BCD_1E0_1_R
- U13 pad 6: BCD_1E1_8_R -> BCD_1E0_8_R
- U14 pad 11: ISO_GND -> DATA_CAN_CHANGE_R
- U14 pad 12: ISO_+5V -> OVERLOAD_R
- U14 pad 13: ISO_GND -> ISO_+5V
- U14 pad 3: BCD_1E6_1_R -> ISO_GND
- U14 pad 4: OVERLOAD_R -> ISO_GND
- U14 pad 5: DATA_CAN_CHANGE_R -> BCD_1E6_1_R
- U15 pad 1: RATIO_N -> INTEG_1
- U15 pad 15: LOCKOUT_N -> AUTORANGE_INH
- U15 pad 2: FUNC_CMD_42 -> INTEG_2
- U15 pad 3: FUNC_CMD_43 -> INTEG_4
- U15 pad 4: INTEG_1 -> FUNC_CMD_43
- U15 pad 5: INTEG_2 -> FUNC_CMD_42
- U15 pad 6: INTEG_4 -> RATIO_N
- U15 pad 7: AUTORANGE_INH -> LOCKOUT_N
- U16 pad 1: RANGE_CMD_2 -> __NOCONNECT
- U16 pad 15: RANGE_CMD_1 -> LED_REMOTE
- U16 pad 2: RANGE_CMD_4 -> __NOCONNECT
- U16 pad 3: SAMPLE_PULSE -> SAMPLE_CONTACT_DRV
- U16 pad 4: SAMPLE_CONTACT_DRV -> RANGE_CMD_4
- U16 pad 5: LED_REMOTE -> RANGE_CMD_2
- U16 pad 6: __NOCONNECT -> SAMPLE_PULSE
- U16 pad 7: __NOCONNECT -> RANGE_CMD_1

Commit message: skidl: swap pins between parts and move the meter-side registers
scripts/optimise_layout.py extends the pin-swap search across parts (any
meter output on any array channel and 74HCT165 input, any command input on
any 74HC595 output) and lets the registers change places and turn 180
degrees; it also scores the clock, latch, /OE, MOSI and chain nets. Result:
all seven registers turned 180 degrees (control and supply pins away from J1
and the arrays), the 74HCT165s in chain order along the bottom row, U15/U16
swapped, decoupling caps moved with the supply pins. Re-routed:

  J1 -> arrays:     102 -> 10 crossings, 481 -> 255 mm of track, 18 -> 6 vias
  74HC595s -> J1:     8 -> 1 crossing,   205 -> 137 mm, 11 -> 7 vias
  control + chains:                      558 -> 494 mm
  whole board:      2227 -> 1868 mm of track, 260 -> 243 vias

DRC, ERC and schematic parity are clean. README bit maps and the routing
review section are updated; the link check is now 1010 on U14 D3..D0.

Co-Authored-By: Claude Opus 5.5 <noreply@anthropic.com>
Claude-Session: https://claude.ai/code/session_01ERGgANCwEg9niX4WLDjBj2
Connections:
- RN1 pad 1: FUNC_OUT_B -> RANGE_OUT_2
- RN1 pad 2: FUNC_OUT_A -> FUNC_OUT_B
- RN1 pad 4: POL_POS -> FUNC_OUT_A
- RN1 pad 5: POL_POS_R -> FUNC_OUT_A_R
- RN1 pad 7: FUNC_OUT_A_R -> FUNC_OUT_B_R
- RN1 pad 8: FUNC_OUT_B_R -> RANGE_OUT_2_R
- RN2 pad 1: PRINT_PULSE -> BCD_1E3_4
- RN2 pad 2: RANGE_OUT_1 -> BCD_1E3_8
- RN2 pad 3: RANGE_OUT_2 -> POL_POS
- RN2 pad 4: RANGE_OUT_4 -> BCD_1E4_1
- RN2 pad 5: RANGE_OUT_4_R -> BCD_1E4_1_R
- RN2 pad 6: RANGE_OUT_2_R -> POL_POS_R
- RN2 pad 7: RANGE_OUT_1_R -> BCD_1E3_8_R
- RN2 pad 8: PRINT_PULSE_R -> BCD_1E3_4_R
- RN3 pad 1: BCD_1E3_1 -> BCD_1E2_1
- RN3 pad 2: BCD_1E3_2 -> PRINT_PULSE
- RN3 pad 3: BCD_1E3_4 -> BCD_1E2_2
- RN3 pad 4: BCD_1E3_8 -> RANGE_OUT_1
- RN3 pad 5: BCD_1E3_8_R -> RANGE_OUT_1_R
- RN3 pad 6: BCD_1E3_4_R -> BCD_1E2_2_R
- RN3 pad 7: BCD_1E3_2_R -> PRINT_PULSE_R
- RN3 pad 8: BCD_1E3_1_R -> BCD_1E2_1_R
- RN4 pad 1: BCD_1E2_1 -> BCD_1E2_4
- RN4 pad 2: BCD_1E2_2 -> BCD_1E2_8
- RN4 pad 3: BCD_1E2_4 -> RANGE_OUT_4
- RN4 pad 4: BCD_1E2_8 -> BCD_1E3_2
- RN4 pad 5: BCD_1E2_8_R -> BCD_1E3_2_R
- RN4 pad 6: BCD_1E2_4_R -> RANGE_OUT_4_R
- RN4 pad 7: BCD_1E2_2_R -> BCD_1E2_8_R
- RN4 pad 8: BCD_1E2_1_R -> BCD_1E2_4_R
- RN5 pad 1: BCD_1E5_1 -> BCD_1E0_1
- RN5 pad 2: BCD_1E5_2 -> BCD_1E4_2
- RN5 pad 3: BCD_1E5_4 -> BCD_1E4_4
- RN5 pad 4: BCD_1E5_8 -> BCD_1E0_4
- RN5 pad 5: BCD_1E5_8_R -> BCD_1E0_4_R
- RN5 pad 6: BCD_1E5_4_R -> BCD_1E4_4_R
- RN5 pad 7: BCD_1E5_2_R -> BCD_1E4_2_R
- RN5 pad 8: BCD_1E5_1_R -> BCD_1E0_1_R
- RN6 pad 1: BCD_1E4_1 -> BCD_1E4_8
- RN6 pad 2: BCD_1E4_2 -> BCD_1E0_8
- RN6 pad 3: BCD_1E4_4 -> BCD_1E1_1
- RN6 pad 4: BCD_1E4_8 -> DATA_CAN_CHANGE
- RN6 pad 5: BCD_1E4_8_R -> DATA_CAN_CHANGE_R
- RN6 pad 6: BCD_1E4_4_R -> BCD_1E1_1_R
- RN6 pad 7: BCD_1E4_2_R -> BCD_1E0_8_R
- RN6 pad 8: BCD_1E4_1_R -> BCD_1E4_8_R
- RN7 pad 1: BCD_1E1_1 -> BCD_1E5_2
- RN7 pad 3: BCD_1E1_4 -> BCD_1E5_4
- RN7 pad 4: BCD_1E1_8 -> BCD_1E1_4
- RN7 pad 5: BCD_1E1_8_R -> BCD_1E1_4_R
- RN7 pad 6: BCD_1E1_4_R -> BCD_1E5_4_R
- RN7 pad 8: BCD_1E1_1_R -> BCD_1E5_2_R
- RN8 pad 1: BCD_1E0_1 -> BCD_1E5_8
- RN8 pad 2: BCD_1E0_2 -> BCD_1E1_8
- RN8 pad 3: BCD_1E0_4 -> BCD_1E6_1
- RN8 pad 4: BCD_1E0_8 -> PRINT_LEVEL
- RN8 pad 5: BCD_1E0_8_R -> PRINT_LEVEL_R
- RN8 pad 6: BCD_1E0_4_R -> BCD_1E6_1_R
- RN8 pad 7: BCD_1E0_2_R -> BCD_1E1_8_R
- RN8 pad 8: BCD_1E0_1_R -> BCD_1E5_8_R
- RN9 pad 1: PRINT_LEVEL -> BCD_1E5_1
- RN9 pad 2: BCD_1E6_1 -> OVERLOAD
- RN9 pad 3: DATA_CAN_CHANGE -> BCD_1E0_2
- RN9 pad 4: OVERLOAD -> BCD_1E3_1
- RN9 pad 5: OVERLOAD_R -> BCD_1E3_1_R
- RN9 pad 6: DATA_CAN_CHANGE_R -> BCD_1E0_2_R
- RN9 pad 7: BCD_1E6_1_R -> OVERLOAD_R
- RN9 pad 8: PRINT_LEVEL_R -> BCD_1E5_1_R
- U10 pad 11: POL_POS_R -> BCD_1E2_8_R
- U10 pad 12: FUNC_OUT_B_R -> BCD_1E2_4_R
- U10 pad 13: FUNC_OUT_A_R -> RANGE_OUT_4_R
- U10 pad 14: POL_NEG_R -> BCD_1E3_2_R
- U10 pad 3: RANGE_OUT_1_R -> BCD_1E2_1_R
- U10 pad 4: PRINT_PULSE_R -> RANGE_OUT_1_R
- U10 pad 5: RANGE_OUT_2_R -> PRINT_PULSE_R
- U10 pad 6: RANGE_OUT_4_R -> BCD_1E2_2_R
- U11 pad 11: BCD_1E3_1_R -> BCD_1E3_8_R
- U11 pad 12: BCD_1E3_8_R -> POL_POS_R
- U11 pad 13: BCD_1E3_2_R -> BCD_1E3_4_R
- U11 pad 14: BCD_1E3_4_R -> BCD_1E4_1_R
- U11 pad 3: BCD_1E2_4_R -> FUNC_OUT_A_R
- U11 pad 4: BCD_1E2_2_R -> RANGE_OUT_2_R
- U11 pad 5: BCD_1E2_1_R -> POL_NEG_R
- U11 pad 6: BCD_1E2_8_R -> FUNC_OUT_B_R
- U12 pad 11: BCD_1E5_1_R -> BCD_1E1_1_R
- U12 pad 12: BCD_1E5_8_R -> BCD_1E0_8_R
- U12 pad 13: BCD_1E5_4_R -> BCD_1E4_8_R
- U12 pad 14: BCD_1E5_2_R -> DATA_CAN_CHANGE_R
- U12 pad 3: BCD_1E4_2_R -> BCD_1E0_1_R
- U12 pad 4: BCD_1E4_4_R -> BCD_1E0_4_R
- U12 pad 5: BCD_1E4_8_R -> BCD_1E4_2_R
- U12 pad 6: BCD_1E4_1_R -> BCD_1E4_4_R
- U13 pad 11: BCD_1E1_1_R -> BCD_1E6_1_R
- U13 pad 13: BCD_1E1_2_R -> BCD_1E5_8_R
- U13 pad 14: BCD_1E1_4_R -> PRINT_LEVEL_R
- U13 pad 3: BCD_1E0_4_R -> BCD_1E1_4_R
- U13 pad 4: BCD_1E0_2_R -> BCD_1E5_2_R
- U13 pad 5: BCD_1E0_1_R -> BCD_1E1_2_R
- U13 pad 6: BCD_1E0_8_R -> BCD_1E5_4_R
- U14 pad 11: DATA_CAN_CHANGE_R -> ISO_GND
- U14 pad 12: OVERLOAD_R -> ISO_+5V
- U14 pad 13: ISO_+5V -> ISO_GND
- U14 pad 3: ISO_GND -> BCD_1E0_2_R
- U14 pad 4: ISO_GND -> OVERLOAD_R
- U14 pad 5: BCD_1E6_1_R -> BCD_1E3_1_R
- U14 pad 6: PRINT_LEVEL_R -> BCD_1E5_1_R
- U15 pad 15: AUTORANGE_INH -> INTEG_4
- U15 pad 2: INTEG_2 -> AUTORANGE_INH
- U15 pad 3: INTEG_4 -> INTEG_2
- U15 pad 4: FUNC_CMD_43 -> RANGE_CMD_1
- U15 pad 5: FUNC_CMD_42 -> RANGE_CMD_2
- U15 pad 6: RATIO_N -> RANGE_CMD_4
- U15 pad 7: LOCKOUT_N -> LED_REMOTE
- U16 pad 1: __NOCONNECT -> RATIO_N
- U16 pad 15: LED_REMOTE -> SAMPLE_CONTACT_DRV
- U16 pad 2: __NOCONNECT -> FUNC_CMD_42
- U16 pad 3: SAMPLE_CONTACT_DRV -> SAMPLE_PULSE
- U16 pad 4: RANGE_CMD_4 -> FUNC_CMD_43
- U16 pad 5: RANGE_CMD_2 -> LOCKOUT_N
- U16 pad 6: SAMPLE_PULSE -> __NOCONNECT
- U16 pad 7: RANGE_CMD_1 -> __NOCONNECT
